Commit message: go to Moai

File: piper_description/urdf/piper_no_gripper_description.urdf (robot description, URDF)
Before this commit: robot piper, 7 links, 6 joints
Joints:
- joint joint1: limit lower=-2.618 upper=2.168 effort=100 velocity=5 -> lower=-2.618 upper=2.618 effort=100 velocity=5
- joint joint2: limit lower=0 upper=3.14 effort=100 velocity=5 -> lower=0 upper=3.3 effort=100 velocity=5
- joint joint6: limit lower=-2.0944 upper=2.0944 effort=100 velocity=5 -> lower=-2.05 upper=2.18 effort=100 velocity=5
