Commit message: 성공은함

File: debug/piper_no_gripper_description.urdf (robot description, URDF)
Before this commit: robot piper, 7 links, 6 joints
Links:
- added link dummy_link
- link link6: mass 0.00699089613564366 -> 0.007
Joints:
- added joint base_to_dummy: type fixed, parent dummy_link, child base_link, origin xyz=0 0 0 rpy=0 0 0
- joint joint1: limit lower=-2.618 upper=2.168 effort=100 velocity=5 -> lower=-2.618 upper=2.618 effort=100 velocity=5
- joint joint6: limit lower=-2.0944 upper=2.0944 effort=100 velocity=5 -> lower=-2.0944 upper=2.0944 effort=100 velocity=3
